File: Plain48/mount.kicad_sch (KiCad schematic)
At the start: 24 parts

Commit message: upd
Parts:
- added H25, H26, H27, H28, H29, H30, H31, H32, H33, H34, H35, H36, H37, H38, H39, H40, H41, H42, H43, H44: MountingHole_Pad, MountingHole:MountingHole_2.2mm_M2_DIN965_Pad, symbol Mechanical:MountingHole_Pad
Connections:
- net GND: now also H25.1, H26.1, H27.1, H28.1, H29.1, H30.1, H31.1, H32.1, H33.1, H34.1, H35.1, H36.1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
