File: Plain48/Plain48.kicad_pcb (KiCad board)
At the start: 2 copper layers, 228.6 x 76.2 mm, 96 parts, among them SW1 SW_Push, SW10 SW_Push, SW11 SW_Push, SW12 SW_Push, SW13 SW_Push, SW14 SW_Push, SW15 SW_Push, SW16 SW_Push, SW17 SW_Push, SW18 SW_Push, SW19 SW_Push, SW2 SW_Push, SW20 SW_Push, SW21 SW_Push, SW22 SW_Push, SW23 SW_Push, SW24 SW_Push, SW25 SW_Push, SW26 SW_Push, SW27 SW_Push, SW28 SW_Push, SW29 SW_Push, SW3 SW_Push, SW30 SW_Push, SW31 SW_Push, SW32 SW_Push, SW33 SW_Push, SW34 SW_Push, SW35 SW_Push, SW36 SW_Push, SW37 SW_Push, SW38 SW_Push, SW39 SW_Push, SW4 SW_Push, SW40 SW_Push, SW41 SW_Push, SW42 SW_Push, SW43 SW_Push, SW44 SW_Push, SW45 SW_Push, SW46 SW_Push, SW47 SW_Push, SW48 SW_Push, SW5 SW_Push, SW6 SW_Push, SW7 SW_Push, SW8 SW_Push, SW9 SW_Push

Commit message: upd
Parts:
- added A1: RaspberryPi_Pico, Module:RaspberryPi_Pico_SMD_HandSolder, F.Cu at (154.3, 67.4)
- added H1: MountingHole_Pad, MountingHole:MountingHole_2.2mm_M2_DIN965_Pad, F.Cu at (47.6, 47.6)
- added H10: MountingHole_Pad, MountingHole:MountingHole_2.2mm_M2_DIN965_Pad, F.Cu at (261.0, 66.7)
- added H11: MountingHole_Pad, MountingHole:MountingHole_2.2mm_M2_DIN965_Pad, F.Cu at (184.8, 85.7)
- added H12: MountingHole_Pad, MountingHole:MountingHole_2.2mm_M2_DIN965_Pad, F.Cu at (261.0, 85.7)
- added H13: MountingHole_Pad, MountingHole:MountingHole_2.2mm_M2_DIN965_Pad, F.Cu at (117.5, 140.7)
- added H14: MountingHole_Pad, MountingHole:MountingHole_2.2mm_M2_DIN965_Pad, F.Cu at (117.5, 146.1)
- added H15: MountingHole_Pad, MountingHole:MountingHole_2.2mm_M2_DIN965_Pad, F.Cu at (117.5, 151.4)
- added H16: MountingHole_Pad, MountingHole:MountingHole_2.2mm_M2_DIN965_Pad, F.Cu at (122.9, 140.7)
- added H17: MountingHole_Pad, MountingHole:MountingHole_2.2mm_M2_DIN965_Pad, F.Cu at (122.9, 146.1)
- added H18: MountingHole_Pad, MountingHole:MountingHole_2.2mm_M2_DIN965_Pad, F.Cu at (122.9, 151.4)
- added H19: MountingHole_Pad, MountingHole:MountingHole_2.2mm_M2_DIN965_Pad, F.Cu at (128.2, 140.7)
- added H2: MountingHole_Pad, MountingHole:MountingHole_2.2mm_M2_DIN965_Pad, F.Cu at (123.8, 47.6)
- added H20: MountingHole_Pad, MountingHole:MountingHole_2.2mm_M2_DIN965_Pad, F.Cu at (128.2, 146.1)
- added H21: MountingHole_Pad, MountingHole:MountingHole_2.2mm_M2_DIN965_Pad, F.Cu at (128.2, 151.4)
- added H22: MountingHole_Pad, MountingHole:MountingHole_2.2mm_M2_DIN965_Pad, F.Cu at (133.6, 140.7)
- added H23: MountingHole_Pad, MountingHole:MountingHole_2.2mm_M2_DIN965_Pad, F.Cu at (133.6, 146.1)
- added H24: MountingHole_Pad, MountingHole:MountingHole_2.2mm_M2_DIN965_Pad, F.Cu at (133.6, 151.4)
- added H3: MountingHole_Pad, MountingHole:MountingHole_2.2mm_M2_DIN965_Pad, F.Cu at (47.6, 66.7)
- added H4: MountingHole_Pad, MountingHole:MountingHole_2.2mm_M2_DIN965_Pad, F.Cu at (123.8, 66.7)
- added H5: MountingHole_Pad, MountingHole:MountingHole_2.2mm_M2_DIN965_Pad, F.Cu at (47.6, 85.7)
- added H6: MountingHole_Pad, MountingHole:MountingHole_2.2mm_M2_DIN965_Pad, F.Cu at (123.8, 85.7)
- added H7: MountingHole_Pad, MountingHole:MountingHole_2.2mm_M2_DIN965_Pad, F.Cu at (184.8, 47.6)
- added H8: MountingHole_Pad, MountingHole:MountingHole_2.2mm_M2_DIN965_Pad, F.Cu at (261.0, 47.6)
- added H9: MountingHole_Pad, MountingHole:MountingHole_2.2mm_M2_DIN965_Pad, F.Cu at (184.8, 66.7)
- D1, D10, D11, D12, D13, D14, D15, D16, D17, D18, D19, D2, D20, D21, D22, D23, D24, D25, D26, D27, D28, D29, D3, D30, D31, D32, D33, D34, D35, D36, D37, D38, D39, D4, D40, D41, D42, D43, D44, D45, D46, D47, D48, D5, D6, D7, D8, D9: moved to F.Cu
- moved SW11 22.9 mm to (251.5, 38.1), turned to 180 degrees
- moved SW20 22.9 mm to (194.3, 57.1), turned to 180 degrees
- moved SW21 22.9 mm to (213.4, 57.1), turned to 180 degrees
- moved SW23 22.9 mm to (251.5, 57.1), turned to 180 degrees
- moved SW32 22.9 mm to (194.3, 76.2), turned to 180 degrees
- moved SW33 22.9 mm to (213.4, 76.2), turned to 180 degrees
- moved SW35 22.9 mm to (251.5, 76.2), turned to 180 degrees
- moved SW44 22.9 mm to (194.3, 95.2), turned to 180 degrees
- moved SW45 22.9 mm to (213.4, 95.2), turned to 180 degrees
- moved SW47 22.9 mm to (251.5, 95.2), turned to 180 degrees
- moved SW8 22.9 mm to (194.3, 38.1), turned to 180 degrees
- moved SW9 22.9 mm to (213.4, 38.1), turned to 180 degrees
- moved SW10 22.9 mm to (232.4, 38.1), turned to 180 degrees
- moved SW12 22.9 mm to (270.5, 38.1), turned to 180 degrees
- moved SW19 22.9 mm to (175.3, 57.1), turned to 180 degrees
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Routing:
- net Col12: track 0.00 -> 225.5 mm
- net Col11: track 0.00 -> 207.2 mm
- net Col10: track 0.00 -> 189.8 mm
- net Col1: track 0.00 -> 178.9 mm
- net Row4: track 419.1 -> 243.0 mm, vias 0 -> 1
- net Row3: track 419.1 -> 246.5 mm, vias 0 -> 1
- net Col9: track 0.00 -> 165.5 mm
- net Col2: track 0.00 -> 161.9 mm
- net Row2: track 419.1 -> 258.7 mm, vias 0 -> 1
- net Col8: track 0.00 -> 150.7 mm
- net Col3: track 0.00 -> 144.9 mm
- net Row1: track 419.1 -> 275.6 mm, vias 0 -> 1
- net Col4: track 0.00 -> 127.6 mm
- net Col5: track 0.00 -> 102.3 mm
- net Col7: track 0.00 -> 77.1 mm
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- added copper zone on B.Cu, net GND
- added copper zone on F.Cu, net GND
Other:
- board size 228.6 x 76.2 mm -> 251.5 x 76.2 mm

Commit message: upd
Parts:
- added H25: MountingHole_Pad, MountingHole:MountingHole_2.2mm_M2_DIN965_Pad, F.Cu at (47.6, 25.1)
- added H26: MountingHole_Pad, MountingHole:MountingHole_2.2mm_M2_DIN965_Pad, F.Cu at (66.7, 25.1)
- added H27: MountingHole_Pad, MountingHole:MountingHole_2.2mm_M2_DIN965_Pad, F.Cu at (85.7, 25.1)
- added H28: MountingHole_Pad, MountingHole:MountingHole_2.2mm_M2_DIN965_Pad, F.Cu at (104.8, 25.1)
- added H29: MountingHole_Pad, MountingHole:MountingHole_2.2mm_M2_DIN965_Pad, F.Cu at (123.8, 25.1)
- added H30: MountingHole_Pad, MountingHole:MountingHole_2.2mm_M2_DIN965_Pad, F.Cu at (184.8, 25.1)
- added H31: MountingHole_Pad, MountingHole:MountingHole_2.2mm_M2_DIN965_Pad, F.Cu at (203.8, 25.1)
- added H32: MountingHole_Pad, MountingHole:MountingHole_2.2mm_M2_DIN965_Pad, F.Cu at (222.9, 25.1)
- added H33: MountingHole_Pad, MountingHole:MountingHole_2.2mm_M2_DIN965_Pad, F.Cu at (241.9, 25.1)
- added H34: MountingHole_Pad, MountingHole:MountingHole_2.2mm_M2_DIN965_Pad, F.Cu at (261.0, 25.1)
- added H35: MountingHole_Pad, MountingHole:MountingHole_2.2mm_M2_DIN965_Pad, F.Cu at (47.6, 108.3)
- added H36: MountingHole_Pad, MountingHole:MountingHole_2.2mm_M2_DIN965_Pad, F.Cu at (66.7, 108.3)
- added H37: MountingHole_Pad, MountingHole:MountingHole_2.2mm_M2_DIN965_Pad, F.Cu at (85.7, 108.3)
- added H38: MountingHole_Pad, MountingHole:MountingHole_2.2mm_M2_DIN965_Pad, F.Cu at (104.8, 108.3)
- added H39: MountingHole_Pad, MountingHole:MountingHole_2.2mm_M2_DIN965_Pad, F.Cu at (123.8, 108.3)
- added H40: MountingHole_Pad, MountingHole:MountingHole_2.2mm_M2_DIN965_Pad, F.Cu at (184.8, 108.3)
- added H41: MountingHole_Pad, MountingHole:MountingHole_2.2mm_M2_DIN965_Pad, F.Cu at (203.8, 108.3)
- added H42: MountingHole_Pad, MountingHole:MountingHole_2.2mm_M2_DIN965_Pad, F.Cu at (222.9, 108.3)
- added H43: MountingHole_Pad, MountingHole:MountingHole_2.2mm_M2_DIN965_Pad, F.Cu at (241.9, 108.3)
- added H44: MountingHole_Pad, MountingHole:MountingHole_2.2mm_M2_DIN965_Pad, F.Cu at (261.0, 108.3)
- moved H21 153.9 mm to (241.9, 47.6)
- moved H20 136.5 mm to (222.9, 47.6)
- moved H24 126.7 mm to (241.9, 85.7)
- moved H19 119.9 mm to (203.8, 47.6)
- moved H23 107.8 mm to (222.9, 85.7)
- moved H13 106.1 mm to (66.7, 47.6)
- moved H15 104.6 mm to (104.8, 47.6)
- moved H14 103.4 mm to (85.7, 47.6)
- moved H22 89.2 mm to (203.8, 85.7)
- moved H16 78.6 mm to (66.7, 85.7)
- moved H17 70.9 mm to (85.7, 85.7)
- moved H18 68.1 mm to (104.8, 85.7)
Routing:
- net Row1: track 275.6 -> 276.1 mm
- net GND: vias 28 -> 13
Other:
- board size 251.5 x 76.2 mm -> 251.5 x 88.2 mm

Commit message: upd
Parts:
- moved H35 0.50 mm to (47.6, 107.8)
- moved H36 0.50 mm to (66.7, 107.8)
- moved H37 0.50 mm to (85.7, 107.8)
- moved H38 0.50 mm to (104.8, 107.8)
- moved H39 0.50 mm to (123.8, 107.8)
Routing:
- net GND: vias 13 -> 15
Other:
- outline, holes or cut-outs redrawn
Changed lines of the file:
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@@
 	(footprint "MountingHole:MountingHole_2.2mm_M2_DIN965_Pad"
 		(layer "F.Cu")
-		(at 66.675 108.28)
+		(at 66.675 107.78)
 		(descr "Mounting Hole 2.2mm, M2, generated by kicad-footprint-generator mountinghole.py")
 		(tags "mountinghole M2 DIN965")
@@
 	(footprint "MountingHole:MountingHole_2.2mm_M2_DIN965_Pad"
 		(layer "F.Cu")
-		(at 85.725 108.28)
+		(at 85.725 107.78)
 		(descr "Mounting Hole 2.2mm, M2, generated by kicad-footprint-generator mountinghole.py")
 		(tags "mountinghole M2 DIN965")
@@
 	(footprint "MountingHole:MountingHole_2.2mm_M2_DIN965_Pad"
 		(layer "F.Cu")
-		(at 47.625 108.28)
+		(at 47.625 107.78)
 		(descr "Mounting Hole 2.2mm, M2, generated by kicad-footprint-generator mountinghole.py")
 		(tags "mountinghole M2 DIN965")
@@
 	(footprint "MountingHole:MountingHole_2.2mm_M2_DIN965_Pad"
 		(layer "F.Cu")
-		(at 123.825 108.28)
+		(at 123.825 107.78)
 		(descr "Mounting Hole 2.2mm, M2, generated by kicad-footprint-generator mountinghole.py")
 		(tags "mountinghole M2 DIN965")
@@
 	(footprint "MountingHole:MountingHole_2.2mm_M2_DIN965_Pad"
 		(layer "F.Cu")
-		(at 241.935 25.08)
+		(at 241.935 25.075)
 		(descr "Mounting Hole 2.2mm, M2, generated by kicad-footprint-generator mountinghole.py")
 		(tags "mountinghole M2 DIN965")
@@
 	(footprint "MountingHole:MountingHole_2.2mm_M2_DIN965_Pad"
 		(layer "F.Cu")
-		(at 104.775 108.28)
+		(at 104.775 107.78)
 		(descr "Mounting Hole 2.2mm, M2, generated by kicad-footprint-generator mountinghole.py")
 		(tags "mountinghole M2 DIN965")
@@
 	(footprint "MountingHole:MountingHole_2.2mm_M2_DIN965_Pad"
 		(layer "F.Cu")
-		(at 260.985 25.08)
+		(at 260.985 25.075)
 		(descr "Mounting Hole 2.2mm, M2, generated by kicad-footprint-generator mountinghole.py")
 		(tags "mountinghole M2 DIN965")
@@
 	(footprint "MountingHole:MountingHole_2.2mm_M2_DIN965_Pad"
 		(layer "F.Cu")
-		(at 222.885 25.08)
+		(at 222.885 25.075)
 		(descr "Mounting Hole 2.2mm, M2, generated by kicad-footprint-generator mountinghole.py")
 		(tags "mountinghole M2 DIN965")
@@
 	(footprint "MountingHole:MountingHole_2.2mm_M2_DIN965_Pad"
 		(layer "F.Cu")
-		(at 184.785 25.08)
+		(at 184.785 25.075)
 		(descr "Mounting Hole 2.2mm, M2, generated by kicad-footprint-generator mountinghole.py")
 		(tags "mountinghole M2 DIN965")
@@
 	(footprint "MountingHole:MountingHole_2.2mm_M2_DIN965_Pad"
 		(layer "F.Cu")
-		(at 203.835 25.08)
+		(at 203.835 25.075)
 		(descr "Mounting Hole 2.2mm, M2, generated by kicad-footprint-generator mountinghole.py")
 		(tags "mountinghole M2 DIN965")
@@
 		(layer "Edge.Cuts")
 	)
+	(gr_arc
+		(start 121.825 104.779978)
+		(mid 122.075011 105.029989)
+		(end 121.825 105.28)
+		(stroke
+			(width 0.05)
+			(type default)
+		)
+		(layer "Edge.Cuts")
+	)
 	(gr_line
 		(start 28.575 102.775)
@@
 	)
 	(gr_arc
-		(start 47.625 110.78)
-		(mid 45.857233 110.047767)
-		(end 45.125 108.28)
+		(start 47.625 110.28)
+		(mid 45.857233 109.547767)
+		(end 45.125 107.78)
 		(stroke
 			(width 0.05)
@@
 	)
 	(gr_line
-		(start 85.725 105.78)
-		(end 122.825 105.78)
+		(start 85.725 105.28)
+		(end 121.825 105.28)
 		(stroke
 			(width 0.05)
@@
 	)
 	(gr_arc
-		(start 123.825 105.78)
-		(mid 125.592767 106.512233)
-		(end 126.325 108.28)
+		(start 123.825 105.28)
+		(mid 125.592767 106.012233)
+		(end 126.325 107.78)
 		(stroke
 			(width 0.05)
@@
 	)
 	(gr_arc
-		(start 126.325 108.28)
-		(mid 125.592767 110.047767)
-		(end 123.825 110.78)
+		(start 126.325 107.78)
+		(mid 125.592767 109.547767)
+		(end 123.825 110.28)
+		(stroke
+			(width 0.05)
+			(type default)
+		)
+		(layer "Edge.Cuts")
+	)
+	(gr_arc
+		(start 123.825 105.28)
+		(mid 123.574989 105.029989)
+		(end 123.825 104.779978)
 		(stroke
 			(width 0.05)
@@
 	)
 	(gr_arc
-		(start 184.785 27.58)
-		(mid 183.017233 26.847767)
-		(end 182.285 25.08)
+		(start 184.785 27.575)
+		(mid 183.017233 26.842767)
+		(end 182.285 25.075)
 		(stroke
 			(width 0.05)
@@
 	)
 	(gr_arc
-		(start 45.125 108.28)
-		(mid 45.857233 106.512233)
-		(end 47.625 105.78)
+		(start 45.125 107.78)
+		(mid 45.857233 106.012233)
+		(end 47.625 105.28)
 		(stroke
 			(width 0.05)
@@
 	)
 	(gr_line
-		(start 123.825 105.78)
-		(end 141.830734 105.78)
+		(start 123.825 104.779978)
+		(end 141.830734 104.774987)
 		(stroke
 			(width 0.05)
@@
 	)
 	(gr_line
-		(start 123.825 110.78)
-		(end 47.625 110.78)
+		(start 123.825 110.28)
+		(end 47.625 110.28)
 		(stroke
 			(width 0.05)
@@
 	)
 	(gr_line
-		(start 141.830734 104.774987)
+		(start 121.825 104.779978)
 		(end 30.575 104.775)
 		(stroke
@@
 	)
 	(gr_arc
-		(start 263.485 25.08)
-		(mid 262.752767 26.847767)
-		(end 260.985 27.58)
+		(start 263.485 25.075)
+		(mid 262.752767 26.842767)
+		(end 260.985 27.575)
 		(stroke
 			(width 0.05)
@@
 	)
 	(gr_arc
-		(start 182.285 25.08)
-		(mid 183.017233 23.312233)
-		(end 184.785 22.58)
+		(start 182.285 25.075)
+		(mid 183.017233 23.307233)
+		(end 184.785 22.575)
 		(stroke
 			(width 0.05)
@@
 	)
 	(gr_line
-		(start 184.785 22.58)
-		(end 260.985 22.58)
+		(start 184.785 22.575)
+		(end 260.985 22.575)
 		(stroke
 			(width 0.05)
@@
 	)
 	(gr_arc
-		(start 260.985 22.58)
-		(mid 262.752767 23.312233)
-		(end 263.485 25.08)
+		(start 260.985 22.575)
+		(mid 262.752767 23.307233)
+		(end 263.485 25.075)
 		(stroke
 			(width 0.05)
@@
 	)
 	(gr_line
-		(start 260.985 27.58)
-		(end 184.785 27.58)
+		(start 260.985 27.575)
+		(end 184.785 27.575)
 		(stroke
 			(width 0.05)
@@
 	)
 	(via
+		(at 123.15 105)
+		(size 0.6)
+		(drill 0.3)
+		(layers "F.Cu" "B.Cu")
+		(free yes)
+		(net 65)
+	)
+	(via
 		(at 176.575 33.475)
 		(size 0.6)
@@
 		(size 0.6)
 		(drill 0.3)
+		(layers "F.Cu" "B.Cu")
+		(free yes)
+		(net 65)
+	)
+	(via
+		(at 122.51 105.01)
+		(size 0.6)
+		(drill 0.3)
